Commit message: Added link for caster wheel and materials

File: urdf/robot.urdf (robot description, URDF)
Before this commit: robot robot, 2 links, 1 joints
Links:
- removed link base_link
- added link link_Right_wheel, mass 1; collision cylinder length=0.12 radius=0.08; collision cylinder length=0.12 radius=0.4
- added link link_caster_wheel, mass 1; collision sphere radius=0.1; collision sphere radius=0.2
- added link link_left_wheel, mass 1; collision cylinder length=0.12 radius=0.08; collision cylinder length=0.12 radius=0.4
Joints:
- removed joint base_to_chassis
- added joint joint_chassis_Right_wheel: type continuous, parent link_chassis, child link_Right_wheel, origin xyz=-0.5 -0.65 0 rpy=0 0 0, axis 0 1 0, limit effort=10000 velocity=1000
- added joint joint_chassis_caster_wheel: type fixed, parent link_chassis, child link_caster_wheel, origin xyz=0.8 0 -0.15 rpy=0 0 0
- added joint joint_chassis_left_wheel: type continuous, parent link_chassis, child link_left_wheel, origin xyz=-0.5 0.65 0 rpy=0 0 0, axis 0 1 0, limit effort=10000 velocity=1000

Commit message: Added meshes for chassis and wheel modified urdf

File: urdf/robot.urdf (robot description, URDF)
Before this commit: robot robot, 4 links, 3 joints
Links:
- link link_Right_wheel: geometry collision cylinder length=0.12 radius=0.08; collision cylinder length=0.12 radius=0.4
- link link_chassis: geometry collision box size=2 1.3 0.4; visual mesh filename=package://robot_description/meshes/chassis.stl
- link link_left_wheel: geometry collision cylinder length=0.12 radius=0.08; collision cylinder length=0.12 radius=0.4

Commit message: added color and friction for links to see in gazebo

File: urdf/robot.urdf (robot description, URDF)
Before this commit: robot robot, 4 links, 3 joints
Links:
- removed link link_Right_wheel
- added link link_right_wheel, mass 1; collision cylinder length=0.12 radius=0.08; collision cylinder length=0.12 radius=0.4
Joints:
- removed joint joint_chassis_Right_wheel
- added joint joint_chassis_right_wheel: type continuous, parent link_chassis, child link_right_wheel, origin xyz=-0.5 -0.65 0 rpy=0 0 0, axis 0 1 0, limit effort=10000 velocity=1000
