Commit message: converted the urdf to xacro file

File: urdf/robot.xacro (robot description, xacro)
@@ -1,78 +1,5 @@
 <?xml version="1.0" ?>
-<robot name="robot">
-    <gazebo reference="link_chassis">
-        <material>Gazebo/BlueGlow</material>
-    </gazebo>
-    <gazebo reference="link_laser_scan">
-        <material>Gazebo/DarkGrey</material>
-    </gazebo>
-    <gazebo reference="link_caster_wheel">
-        <material>Gazebo/DarkGrey</material>
-        <mu1>0</mu1>
-        <mu2>0</mu2>
-    </gazebo>
-    <gazebo reference="link_left_wheel">
-        <material>Gazebo/FlatBlack</material>
-        <mu1>1</mu1>
-        <mu2>1</mu2>
-    </gazebo>
-    <gazebo reference="link_right_wheel">
-        <material>Gazebo/FlatBlack</material>
-        <mu1>1</mu1>
-        <mu2>1</mu2>
-    </gazebo>
-    <gazebo reference="joint_chassis_caster_wheel">
-        <preserveFixedJoint>true
-    </preserveFixedJoint>
-    </gazebo>
-    <gazebo reference="joint_laser_scan_chassis">
-        <preserveFixedJoint>true</preserveFixedJoint>
-    </gazebo>
-    <gazebo>
-    <plugin filename="libgazebo_ros_diff_drive.so" name="differential_drive_controller">
-        <alwaysOn>true</alwaysOn>
-        <updateRate>20</updateRate>
-        <leftJoint>joint_chassis_left_wheel</leftJoint>
-        <rightJoint>joint_chassis_right_wheel</rightJoint>
-        <wheelSeparation>1.66</wheelSeparation>
-        <wheelDiameter>0.8</wheelDiameter>
-        <torque>10</torque>
-        <commandTopic>cmd_vel</commandTopic>
-        <odometryTopic>odom</odometryTopic>
-        <odometryFrame>odom</odometryFrame>
-        <robotBaseFrame>link_chassis</robotBaseFrame>
-    </plugin>
-    </gazebo>
-    <gazebo reference="link_laser_scan">
-        <sensor type="ray" name="head_hokuyo_sensor">
-            <pose>0 0 0 0 0 0</pose>
-            <visualize>true</visualize>
-            <update_rate>20</update_rate>
-            <ray>
-                <scan>
-                    <horizontal>
-                        <samples>720</samples>
-                        <resolution>1</resolution>
-                        <min_angle>-1.570796</min_angle>
-                        <max_angle>1.570796</max_angle>
-                    </horizontal>
-                </scan>
-                <range>
-                    <min>0.20</min>
-                    <max>10.0</max>
-                    <resolution>0.01</resolution>
-                </range>
-                <noise>
-                    <type>gaussian</type>
-                    <mean>0.0</mean>
-                    <stddev>0.01</stddev>
-                </noise>
-            </ray>
-            <plugin name="gazebo_ros_head_hokuyo_controller" filename="libgazebo_ros_laser.so">
-                <topicName>/laser/scan</topicName>
-                <frameName>sensor_laser</frameName>
-            </plugin>
-        </sensor>
-    </gazebo>
+<robot name="robot" xmlns:xacro="http://www.ros.org/wiki/xacro">
+    <xacro:include filename="$(find robot_description)/urdf/robot.gazebo" />
     <!-- Link - chassis -->
     <link name="link_chassis">

Commit message: added math expressions

File: urdf/robot.xacro (robot description, xacro)
@@ -2,8 +2,11 @@
 <robot name="robot" xmlns:xacro="http://www.ros.org/wiki/xacro">
     <xacro:include filename="$(find robot_description)/urdf/robot.gazebo" />
+    <!-- Parameters -->
+    <xacro:property name="chassis_mass" value="10" />
+    <xacro:property name="pi" value="3.1415926" />
     <!-- Link - chassis -->
     <link name="link_chassis">
         <inertial>
-            <mass value="10" />
+            <mass value="${chassis_mass}" />
             <origin xyz="0 0 0.3" rpy="0 0 0" />
             <inertia ixx="1.5417" ixy="0" ixz="0" iyy="3.467" iyz="0" izz="4.742" />
@@ -41,5 +44,5 @@
         <!-- Tires -->
         <collision>
-            <origin rpy="1.5707 0 0" xyz="0 0.18 0" />
+            <origin rpy="${pi/2} 0 0" xyz="0 0.18 0" />
             <geometry>
                 <cylinder length="0.12" radius="0.4"/>
@@ -47,5 +50,5 @@
         </collision>
         <visual>
-            <origin rpy="1.5707 0 0" xyz="0 0.18 0" />
+            <origin rpy="${pi/2} 0 0" xyz="0 0.18 0" />
             <geometry>
                 <mesh filename="package://robot_description/meshes/wheel.stl" />
@@ -57,11 +60,11 @@
         <!-- Axle -->
         <collision>
-            <origin rpy="1.5707 0 0" xyz="0 0.06 0" />
-            <geometry>
-                <cylinder length="0.12" radius="0.08"/>
-            </geometry>
-        </collision>
-        <visual>
-            <origin rpy="1.5707 0 0" xyz="0 0.06 0" />
+            <origin rpy="${pi/2} 0 0" xyz="0 0.06 0" />
+            <geometry>
+                <cylinder length="0.12" radius="0.08"/>
+            </geometry>
+        </collision>
+        <visual>
+            <origin rpy="${pi/2} 0 0" xyz="0 0.06 0" />
             <geometry>
                 <cylinder length="0.12" radius="0.08"/>
@@ -73,5 +76,5 @@
         <!-- Hubcap -->
         <visual>
-            <origin rpy="1.5707 0 0" xyz="0 0.25 0" />
+            <origin rpy="{pi/2} 0 0" xyz="0 0.25 0" />
             <geometry>
                 <box size="0.02 0.5 0.02" />
@@ -100,5 +103,5 @@
         <!-- Tires -->
         <collision>
-            <origin rpy="1.5707 0 0" xyz="0 -0.18 0" />
+            <origin rpy="${pi/2} 0 0" xyz="0 -0.18 0" />
             <geometry>
                 <cylinder length="0.12" radius="0.4"/>
@@ -106,5 +109,5 @@
         </collision>
         <visual>
-            <origin rpy="1.5707 0 0" xyz="0 -0.18 0" />
+            <origin rpy="${pi/2} 0 0" xyz="0 -0.18 0" />
             <geometry>
                 <mesh filename="package://robot_description/meshes/wheel.stl" />
@@ -116,11 +119,11 @@
         <!-- Axle -->
         <collision>
-            <origin rpy="1.5707 0 0" xyz="0 -0.06 0" />
-            <geometry>
-                <cylinder length="0.12" radius="0.08"/>
-            </geometry>
-        </collision>
-        <visual>
-            <origin rpy="1.5707 0 0" xyz="0 -0.06 0" />
+            <origin rpy="${pi/2} 0 0" xyz="0 -0.06 0" />
+            <geometry>
+                <cylinder length="0.12" radius="0.08"/>
+            </geometry>
+        </collision>
+        <visual>
+            <origin rpy="${pi/2} 0 0" xyz="0 -0.06 0" />
             <geometry>
                 <cylinder length="0.12" radius="0.08"/>
@@ -132,5 +135,5 @@
         <!-- Hubcap -->
         <visual>
-            <origin rpy="1.5707 0 0" xyz="0 0.25 0" />
+            <origin rpy="${pi/2} 0 0" xyz="0 0.25 0" />
             <geometry>
                 <box size="0.02 0.5 0.02" />

Commit message: added robot joint control ros plugin

File: urdf/robot.xacro (robot description, xacro)
@@ -221,3 +221,44 @@
         </collision>
     </link>
+    <!-- Joint - Chassis/tail -->
+    <joint name="joint_tail" type="continuous">
+        <origin rpy="0 0 0" xyz="-1 0 0" />
+        <axis rpy="0 0 0" xyz="0 1 0" />
+        <parent link="link_chassis" />
+        <child link="link_tail" />
+        <joint_properties damping="1.0" friction="1.0" />
+    </joint>
+    <!-- link - Robot tail -->
+    <link name="link_tail">
+        <inertial>
+            <origin xyz="0 0 0" rpy="0 0 0" />
+            <mass value="0.5" />
+            <inertia ixx="0.000252666666667" ixy="0" ixz="0" iyy="0.000252666666667" iyz="0" izz="0.0005" />
+        </inertial>
+        <visual>
+            <origin xyz="-0.2 0 0" rpy="0 ${pi/2} 0"/>
+            <geometry>
+                <cylinder radius="0.05" length="0.40"/>
+            </geometry>
+            <material name="Red">
+                <color rgba="0.7 0.1 0.1 1" />
+            </material>
+        </visual>
+        <collision>
+            <origin xyz="-0.2 0 0" rpy="0 ${pi/2} 0"/>
+            <geometry>
+                <cylinder radius="0.05" length="0.40"/>
+            </geometry>
+        </collision>
+    </link>
+    <transmission name="tran_tail">
+        <type>transmission_interface/SimpleTransmission</type>
+        <joint name="joint_tail">
+            <hardwareInterface>hardware_interface/EffortJointInterface</hardwareInterface>
+        </joint>
+        <actuator name="motor_joint_tail">
+            <hardwareInterface>hardware_interface/EffortJointInterface</hardwareInterface>
+            <mechanicalReduction>1</mechanicalReduction>
+        </actuator>
+    </transmission>
 </robot>
